Commit message: gui added, com task control from gui available

File: dyros_red_description/robots/dyros_red_robot (copy).urdf (robot description, URDF)
Before this commit: robot dyros_red_description, 32 links, 31 joints
Links:
- added link base_link
Joints:
- added joint virtual: type floating, parent base_link, child Pelvis_Link, origin xyz=0 0 0 rpy=0 0 0
