Commit message: lower body inertia re-arrangement

File: dyros_red_description/robots/dyros_red_robot.urdf (robot description, URDF)
Before this commit: robot dyros_red_description, 32 links, 31 joints
Links:
- link L_AnkleCenter_Link: mass 0.38954 -> 2.51
- link L_AnkleRoll_Link: mass 0.98346 -> 3.464
- link L_HipCenter_Link: mass 0.37947 -> 2.67
- link L_HipRoll_Link: mass 0.46745 -> 2.679
- link L_Knee_Link: mass 0.70655 -> 3.883
- link L_Thigh_Link: mass 1.0564 -> 5.366
- link R_AnkleCenter_Link: mass 0.38954 -> 2.51
- link R_AnkleRoll_Link: mass 0.98346 -> 3.464
- link R_HipCenter_Link: mass 0.37947 -> 2.67
- link R_HipRoll_Link: mass 0.46745 -> 2.679
- link R_Knee_Link: mass 0.70655 -> 3.883
- link R_Thigh_Link: mass 1.0564 -> 5.366

File: dyros_red_description/robots/dyros_red_robot_origin.urdf (robot description, URDF)
Before this commit: robot dyros_red_description, 33 links, 32 joints
Links:
- removed link base_link
Joints:
- removed joint virtual
