Commit message: Inertial property calib

File: dyros_red_lowerbody_description/robots/red_robot_lowerbody.urdf (robot description, URDF)
Before this commit: robot red_robot, 15 links, 14 joints
Links:
- link AnkleCenter_L_Link: mass 2.51 -> 2.693
- link AnkleCenter_R_Link: mass 2.51 -> 2.693
- link AnkleRoll_L_Link: mass 3.464 -> 3.632
- link AnkleRoll_R_Link: mass 3.464 -> 3.632
- link HipCenter_L_Link: mass 2.67 -> 2.865
- link HipCenter_R_Link: mass 2.67 -> 2.865
- link HipRoll_L_Link: mass 2.679 -> 2.874
- link HipRoll_R_Link: mass 2.679 -> 2.874
- link Knee_L_Link: mass 3.883 -> 4.072
- link Knee_R_Link: mass 3.883 -> 4.072
- link Thigh_L_Link: mass 5.366 -> 5.756
- link Thigh_R_Link: mass 5.366 -> 5.756
